File: src/schemas/rhizome/KiCad/SlimVersionRhizome/SlimRhizz/SlimRhizz.kicad_sch (KiCad schematic)
At the start: 19 parts, among them J1 POWER_IN, J2 WS2812_Tip1, J3 WS2812_Tip2, J4 APA102_Strip, J5 Haptic_DRV1, J6 Haptic_DRV2, J7 Pogo_Male, J8 Pogo_Female, U2 74AHCT125

Commit message: update PCB
Other:
- moved on the sheet: J1, J2, J3, J4, J5, U2E

Commit message: pcb v2
Parts:
- added D1: PWR, LED_SMD:LED_0402_1005Metric, symbol Device:LED_Small
- added D2: HBT, LED_SMD:LED_0402_1005Metric, symbol Device:LED_Small
- added D3: L-Connect, LED_SMD:LED_0402_1005Metric, symbol Device:LED_Small
- added D4: R-Connect, LED_SMD:LED_0402_1005Metric, symbol Device:LED_Small
- added R5: 1000, Resistor_SMD:R_0402_1005Metric, symbol Device:R_Small
- added R6, R7, R8: 330, Resistor_SMD:R_0402_1005Metric, symbol Device:R_Small
- C1, C2, C3: footprint Capacitor_THT:CP_Radial_D10.0mm_P5.00mm -> Capacitor_SMD:CP_Elec_10x10.5
- C4, C5: footprint Capacitor_THT:CP_Radial_D6.3mm_P2.50mm -> Capacitor_SMD:CP_Elec_6.3x5.4
- R1, R2, R4: footprint Resistor_THT:R_Axial_DIN0207_L6.3mm_D2.5mm_P7.62mm_Horizontal -> Resistor_SMD:R_0805_2012Metric
- R3: value 330 -> 220; footprint Resistor_THT:R_Axial_DIN0207_L6.3mm_D2.5mm_P7.62mm_Horizontal -> Resistor_SMD:R_0805_2012Metric
- U2, u1: now left out of the parts list
Connections:
- net +5V: now also R5.2
- net GND: now also D1.1 (K), D2.1 (K), D3.1 (K), D4.1 (K)
- net at u1.2: now also R6.1
- net at u1.3: now also R7.1
- net at u1.4: now also R8.1
- new net: D3.2 (A), R7.2
- new net: D4.2 (A), R8.2
- new net: D2.2 (A), R6.2
- new net: D1.2 (A), R5.1
- no-connect marks 10 -> 7
